Commit message: fix: resolve all critical issues for UR5 Gazebo simulation
- Replace missing mesh files with simple geometry placeholders (cylinders/boxes)
- Fix ros2_control plugin from gz_ros2_control to gazebo_ros2_control
- Fix UR5 kinematics with correct joint axes and DH parameters
- Add missing empty.sdf world file
- Fix spawn_ur5.py parameter passing for robot_description
- Fix SRDF to use tool0 instead of non-existent ee_link
- Fix Dockerfile COPY paths and update dependencies
- Fix CMakeLists.txt to install scripts directory
- Fix package.xml XML format and update dependencies
- Fix MoveIt2 launch file robot_description processing
- Update moveit_controllers.yaml format

Fixes: #19 #20 #21 #22 #23 #24 #25 #26 #27 #28

File: ur5_gazebo_ros2/ur5_description/urdf/ur5.ros2_control.xacro (robot description, xacro)
@@ -1,9 +1,9 @@
 <?xml version="1.0"?>
 <robot xmlns:xacro="http://wiki.ros.org/xacro">
-  <!-- ROS2 Control UR5 -->
+  <!-- ROS2 Control UR5 - Gazebo Classic -->
   <xacro:macro name="ur5_ros2_control" params="name prefix">
     <ros2_control name="${name}" type="system">
       <hardware>
-        <plugin>gz_ros2_control/GazeboSimSystem</plugin>
+        <plugin>gazebo_ros2_control/GazeboSystem</plugin>
       </hardware>
       <joint name="${prefix}shoulder_pan_joint">

File: ur5_gazebo_ros2/ur5_description/urdf/ur5_macro.xacro (robot description, xacro)
@@ -2,5 +2,9 @@
 <robot xmlns:xacro="http://wiki.ros.org/xacro">
   <!--
-    Universal Robots UR5
+    Universal Robots UR5 - Simplified Description
+    Uses basic geometry (cylinders, boxes) as placeholders
+    since official mesh files are not included in this repository.
+    For production use with official UR5 meshes, see:
+    https://github.com/ros-industrial/universal_robot
   -->
   <xacro:macro name="ur5_robot" params="prefix joint_limited
@@ -14,5 +18,8 @@
     safety_limits:=false safety_pos_margin:=0.15
     safety_k_position:=20">
-    <!-- Inertia parameters -->
+    <!-- ============================================================ -->
+    <!-- Physical Parameters (from Universal Robots UR5 specification) -->
+    <!-- ============================================================ -->
+    <!-- Mass (kg) -->
     <xacro:property name="base_mass" value="4.0" />
     <xacro:property name="shoulder_mass" value="3.7000" />
@@ -22,13 +29,19 @@
     <xacro:property name="wrist_2_mass" value="1.2190" />
     <xacro:property name="wrist_3_mass" value="0.1879" />
-    <!-- Link offsets -->
-    <xacro:property name="shoulder_y_offset" value="0.089159" />
-    <xacro:property name="upper_arm_y_offset" value="-0.13625" />
-    <xacro:property name="forearm_y_offset" value="-0.1197" />
-    <xacro:property name="wrist_1_z_offset" value="0.093" />
-    <xacro:property name="wrist_2_z_offset" value="0.0" />
-    <xacro:property name="wrist_3_z_offset" value="0.0" />
-    <xacro:property name="wrist_3_length" value="0.0" />
-    <!-- Joint limits -->
+    <!-- Center of Mass offsets (m) -->
+    <xacro:property name="shoulder_cog" value="0.0 0.0 0.0" />
+    <xacro:property name="upper_arm_cog" value="0.0 -0.13625 0.0" />
+    <xacro:property name="forearm_cog" value="0.0 -0.1197 0.0" />
+    <xacro:property name="wrist_1_cog" value="0.0 0.0 0.093" />
+    <xacro:property name="wrist_2_cog" value="0.0 0.0 0.0" />
+    <xacro:property name="wrist_3_cog" value="0.0 0.0 0.0" />
+    <!-- Link dimensions (m) -->
+    <xacro:property name="shoulder_height" value="0.089159" />
+    <xacro:property name="upper_arm_length" value="0.425" />
+    <xacro:property name="forearm_length" value="0.39225" />
+    <xacro:property name="wrist_1_length" value="0.093" />
+    <xacro:property name="wrist_2_length" value="0.09465" />
+    <xacro:property name="wrist_3_length" value="0.0823" />
+    <!-- Joint velocity limits (rad/s) -->
     <xacro:property name="shoulder_pan_velocity" value="3.15" />
     <xacro:property name="shoulder_lift_velocity" value="3.15" />
@@ -37,14 +50,20 @@
     <xacro:property name="wrist_2_velocity" value="3.2" />
     <xacro:property name="wrist_3_velocity" value="3.2" />
-    <!-- Base link -->
+    <!-- ============================================================ -->
+    <!-- Link Definitions (using simple geometry placeholders) -->
+    <!-- ============================================================ -->
+    <!-- Base Link -->
     <link name="${prefix}base_link">
       <visual>
-        <geometry>
-          <mesh filename="package://ur5_description/meshes/ur5/visual/base.dae"/>
-        </geometry>
-      </visual>
-      <collision>
-        <geometry>
-          <mesh filename="package://ur5_description/meshes/ur5/collision/base.stl"/>
+        <origin xyz="0 0 0" rpy="0 0 0"/>
+        <geometry>
+          <cylinder radius="0.06" length="0.08"/>
+        </geometry>
+        <material name="Grey"/>
+      </visual>
+      <collision>
+        <origin xyz="0 0 0" rpy="0 0 0"/>
+        <geometry>
+          <cylinder radius="0.06" length="0.08"/>
         </geometry>
       </collision>
@@ -55,14 +74,17 @@
       </inertial>
     </link>
-    <!-- Shoulder link -->
+    <!-- Shoulder Link -->
     <link name="${prefix}shoulder_link">
       <visual>
-        <geometry>
-          <mesh filename="package://ur5_description/meshes/ur5/visual/shoulder.dae"/>
-        </geometry>
-      </visual>
-      <collision>
-        <geometry>
-          <mesh filename="package://ur5_description/meshes/ur5/collision/shoulder.stl"/>
+        <origin xyz="0 0 0" rpy="0 0 0"/>
+        <geometry>
+          <cylinder radius="0.075" length="0.12"/>
+        </geometry>
+        <material name="Grey"/>
+      </visual>
+      <collision>
+        <origin xyz="0 0 0" rpy="0 0 0"/>
+        <geometry>
+          <cylinder radius="0.075" length="0.12"/>
         </geometry>
       </collision>
@@ -73,99 +95,119 @@
       </inertial>
     </link>
-    <!-- Upper arm link -->
+    <!-- Upper Arm Link -->
     <link name="${prefix}upper_arm_link">
       <visual>
-        <geometry>
-          <mesh filename="package://ur5_description/meshes/ur5/visual/upperarm.dae"/>
-        </geometry>
-      </visual>
-      <collision>
-        <geometry>
-          <mesh filename="package://ur5_description/meshes/ur5/collision/upperarm.stl"/>
+        <origin xyz="0 -${upper_arm_length/2} 0" rpy="0 0 0"/>
+        <geometry>
+          <box size="0.08 ${upper_arm_length} 0.08"/>
+        </geometry>
+        <material name="Blue"/>
+      </visual>
+      <collision>
+        <origin xyz="0 -${upper_arm_length/2} 0" rpy="0 0 0"/>
+        <geometry>
+          <box size="0.08 ${upper_arm_length} 0.08"/>
         </geometry>
       </collision>
       <inertial>
         <mass value="${upper_arm_mass}"/>
-        <origin xyz="0 ${upper_arm_y_offset} 0" rpy="0 0 0"/>
+        <origin xyz="0 -${upper_arm_length/2} 0" rpy="0 0 0"/>
         <inertia ixx="0.133886" ixy="0.0" ixz="0.0" iyy="0.0151074" iyz="0.0" izz="0.13774"/>
       </inertial>
     </link>
-    <!-- Forearm link -->
+    <!-- Forearm Link -->
     <link name="${prefix}forearm_link">
       <visual>
-        <geometry>
-          <mesh filename="package://ur5_description/meshes/ur5/visual/forearm.dae"/>
-        </geometry>
-      </visual>
-      <collision>
-        <geometry>
-          <mesh filename="package://ur5_description/meshes/ur5/collision/forearm.stl"/>
+        <origin xyz="0 -${forearm_length/2} 0" rpy="0 0 0"/>
+        <geometry>
+          <box size="0.065 ${forearm_length} 0.065"/>
+        </geometry>
+        <material name="Blue"/>
+      </visual>
+      <collision>
+        <origin xyz="0 -${forearm_length/2} 0" rpy="0 0 0"/>
+        <geometry>
+          <box size="0.065 ${forearm_length} 0.065"/>
         </geometry>
       </collision>
       <inertial>
         <mass value="${forearm_mass}"/>
-        <origin xyz="0 ${forearm_y_offset} 0" rpy="0 0 0"/>
+        <origin xyz="0 -${forearm_length/2} 0" rpy="0 0 0"/>
         <inertia ixx="0.0311898" ixy="0.0" ixz="0.0" iyy="0.004095" iyz="0.0" izz="0.0311898"/>
       </inertial>
     </link>
-    <!-- Wrist 1 link -->
+    <!-- Wrist 1 Link -->
     <link name="${prefix}wrist_1_link">
       <visual>
-        <geometry>
-          <mesh filename="package://ur5_description/meshes/ur5/visual/wrist1.dae"/>
-        </geometry>
-      </visual>
-      <collision>
-        <geometry>
-          <mesh filename="package://ur5_description/meshes/ur5/collision/wrist1.stl"/>
+        <origin xyz="0 0 0" rpy="0 0 0"/>
+        <geometry>
+          <cylinder radius="0.04" length="${wrist_1_length}"/>
+        </geometry>
+        <material name="LightGrey"/>
+      </visual>
+      <collision>
+        <origin xyz="0 0 0" rpy="0 0 0"/>
+        <geometry>
+          <cylinder radius="0.04" length="${wrist_1_length}"/>
         </geometry>
       </collision>
       <inertial>
         <mass value="${wrist_1_mass}"/>
-        <origin xyz="0 ${wrist_1_z_offset} 0" rpy="0 0 0"/>
+        <origin xyz="0 0 0" rpy="0 0 0"/>
         <inertia ixx="0.0025599" ixy="0.0" ixz="0.0" iyy="0.000792168" iyz="0.0" izz="0.0025599"/>
       </inertial>
     </link>
-    <!-- Wrist 2 link -->
+    <!-- Wrist 2 Link -->
     <link name="${prefix}wrist_2_link">
       <visual>
-        <geometry>
-          <mesh filename="package://ur5_description/meshes/ur5/visual/wrist2.dae"/>
-        </geometry>
-      </visual>
-      <collision>
-        <geometry>
-          <mesh filename="package://ur5_description/meshes/ur5/collision/wrist2.stl"/>
+        <origin xyz="0 0 0" rpy="0 0 0"/>
+        <geometry>
+          <cylinder radius="0.04" length="${wrist_2_length}"/>
+        </geometry>
+        <material name="LightGrey"/>
+      </visual>
+      <collision>
+        <origin xyz="0 0 0" rpy="0 0 0"/>
+        <geometry>
+          <cylinder radius="0.04" length="${wrist_2_length}"/>
         </geometry>
       </collision>
       <inertial>
         <mass value="${wrist_2_mass}"/>
-        <origin xyz="0 ${wrist_2_z_offset} 0" rpy="0 0 0"/>
+        <origin xyz="0 0 0" rpy="0 0 0"/>
         <inertia ixx="0.0025599" ixy="0.0" ixz="0.0" iyy="0.000792168" iyz="0.0" izz="0.0025599"/>
       </inertial>
     </link>
-    <!-- Wrist 3 link -->
+    <!-- Wrist 3 Link -->
     <link name="${prefix}wrist_3_link">
       <visual>
-        <geometry>
-          <mesh filename="package://ur5_description/meshes/ur5/visual/wrist3.dae"/>
-        </geometry>
-      </visual>
-      <collision>
-        <geometry>
-          <mesh filename="package://ur5_description/meshes/ur5/collision/wrist3.stl"/>
+        <origin xyz="0 0 0" rpy="0 0 0"/>
+        <geometry>
+          <cylinder radius="0.035" length="${wrist_3_length}"/>
+        </geometry>
+        <material name="LightGrey"/>
+      </visual>
+      <collision>
+        <origin xyz="0 0 0" rpy="0 0 0"/>
+        <geometry>
+          <cylinder radius="0.035" length="${wrist_3_length}"/>
         </geometry>
       </collision>
       <inertial>
         <mass value="${wrist_3_mass}"/>
-        <origin xyz="0 ${wrist_3_z_offset} 0" rpy="0 0 0"/>
+        <origin xyz="0 0 0" rpy="0 0 0"/>
         <inertia ixx="0.000132134" ixy="0.0" ixz="0.0" iyy="0.000132134" iyz="0.0" izz="0.00021942"/>
       </inertial>
     </link>
-    <!-- Joints -->
+    <!-- Tool0 Link (End Effector) -->
+    <link name="${prefix}tool0"/>
+    <!-- ============================================================ -->
+    <!-- Joint Definitions -->
+    <!-- ============================================================ -->
+    <!-- Shoulder Pan Joint (revolute around Z) -->
     <joint name="${prefix}shoulder_pan_joint" type="revolute">
       <parent link="${prefix}base_link"/>
       <child link="${prefix}shoulder_link"/>
-      <origin xyz="0 0 0.089159" rpy="0 0 0"/>
+      <origin xyz="0 0 ${shoulder_height}" rpy="0 0 0"/>
       <axis xyz="0 0 1"/>
       <limit lower="${shoulder_pan_lower_limit}" upper="${shoulder_pan_upper_limit}"
@@ -176,10 +218,11 @@
                           k_position="${safety_k_position}" k_velocity="0.0"/>
       </xacro:if>
-      <dynamics damping="0" friction="0"/>
-    </joint>
+      <dynamics damping="0.5" friction="0.5"/>
+    </joint>
+    <!-- Shoulder Lift Joint (revolute around Y) -->
     <joint name="${prefix}shoulder_lift_joint" type="revolute">
       <parent link="${prefix}shoulder_link"/>
       <child link="${prefix}upper_arm_link"/>
-      <origin xyz="0 ${shoulder_y_offset} 0" rpy="0 ${pi/2} 0"/>
+      <origin xyz="0 0 0" rpy="${pi/2} 0 0"/>
       <axis xyz="0 0 1"/>
       <limit lower="${shoulder_lift_lower_limit}" upper="${shoulder_lift_upper_limit}"
@@ -190,10 +233,11 @@
                           k_position="${safety_k_position}" k_velocity="0.0"/>
       </xacro:if>
-      <dynamics damping="0" friction="0"/>
-    </joint>
+      <dynamics damping="0.5" friction="0.5"/>
+    </joint>
+    <!-- Elbow Joint (revolute around Y) -->
     <joint name="${prefix}elbow_joint" type="revolute">
       <parent link="${prefix}upper_arm_link"/>
       <child link="${prefix}forearm_link"/>
-      <origin xyz="0 ${upper_arm_y_offset} 0" rpy="0 0 0"/>
+      <origin xyz="0 -${upper_arm_length} 0" rpy="0 0 0"/>
       <axis xyz="0 0 1"/>
       <limit lower="${elbow_joint_lower_limit}" upper="${elbow_joint_upper_limit}"
@@ -204,10 +248,11 @@
                           k_position="${safety_k_position}" k_velocity="0.0"/>
       </xacro:if>
-      <dynamics damping="0" friction="0"/>
-    </joint>
+      <dynamics damping="0.5" friction="0.5"/>
+    </joint>
+    <!-- Wrist 1 Joint (revolute around Y) -->
     <joint name="${prefix}wrist_1_joint" type="revolute">
       <parent link="${prefix}forearm_link"/>
       <child link="${prefix}wrist_1_link"/>
-      <origin xyz="0 ${forearm_y_offset} 0" rpy="0 0 0"/>
+      <origin xyz="0 -${forearm_length} 0" rpy="${pi/2} 0 0"/>
       <axis xyz="0 0 1"/>
       <limit lower="${wrist_1_lower_limit}" upper="${wrist_1_upper_limit}"
@@ -218,10 +263,11 @@
                           k_position="${safety_k_position}" k_velocity="0.0"/>
       </xacro:if>
-      <dynamics damping="0" friction="0"/>
-    </joint>
+      <dynamics damping="0.5" friction="0.5"/>
+    </joint>
+    <!-- Wrist 2 Joint (revolute around Z) -->
     <joint name="${prefix}wrist_2_joint" type="revolute">
       <parent link="${prefix}wrist_1_link"/>
       <child link="${prefix}wrist_2_link"/>
-      <origin xyz="0 0 ${wrist_1_z_offset}" rpy="0 ${pi/2} 0"/>
+      <origin xyz="0 0 ${wrist_1_length}" rpy="${-pi/2} 0 0"/>
       <axis xyz="0 0 1"/>
       <limit lower="${wrist_2_lower_limit}" upper="${wrist_2_upper_limit}"
@@ -232,10 +278,11 @@
                           k_position="${safety_k_position}" k_velocity="0.0"/>
       </xacro:if>
-      <dynamics damping="0" friction="0"/>
-    </joint>
+      <dynamics damping="0.5" friction="0.5"/>
+    </joint>
+    <!-- Wrist 3 Joint (revolute around Y) -->
     <joint name="${prefix}wrist_3_joint" type="revolute">
       <parent link="${prefix}wrist_2_link"/>
       <child link="${prefix}wrist_3_link"/>
-      <origin xyz="0 0 ${wrist_2_z_offset}" rpy="0 0 0"/>
+      <origin xyz="0 ${wrist_2_length} 0" rpy="${pi/2} 0 0"/>
       <axis xyz="0 0 1"/>
       <limit lower="${wrist_3_lower_limit}" upper="${wrist_3_upper_limit}"
@@ -246,13 +293,53 @@
                           k_position="${safety_k_position}" k_velocity="0.0"/>
       </xacro:if>
-      <dynamics damping="0" friction="0"/>
-    </joint>
-    <!-- Tool frame -->
-    <link name="${prefix}tool0"/>
+      <dynamics damping="0.5" friction="0.5"/>
+    </joint>
+    <!-- Tool0 Joint (fixed) -->
     <joint name="${prefix}tool0_joint" type="fixed">
       <parent link="${prefix}wrist_3_link"/>
       <child link="${prefix}tool0"/>
-      <origin xyz="0 0 ${wrist_3_length}" rpy="0 ${pi/2} ${pi/2}"/>
-    </joint>
+      <origin xyz="0 0 ${wrist_3_length}" rpy="${-pi/2} ${-pi/2} 0"/>
+    </joint>
+    <!-- ============================================================ -->
+    <!-- Gazebo Plugin (using gazebo_ros2_control for Gazebo Classic) -->
+    <!-- ============================================================ -->
+    <xacro:include filename="$(find ur5_description)/urdf/ur5.ros2_control.xacro"/>
+    <xacro:ur5_ros2_control name="UR5Control" prefix=""/>
+    <!-- ============================================================ -->
+    <!-- Gazebo Colors -->
+    <!-- ============================================================ -->
+    <gazebo reference="${prefix}base_link">
+      <material>Gazebo/Grey</material>
+    </gazebo>
+    <gazebo reference="${prefix}shoulder_link">
+      <material>Gazebo/Grey</material>
+    </gazebo>
+    <gazebo reference="${prefix}upper_arm_link">
+      <material>Gazebo/Blue</material>
+    </gazebo>
+    <gazebo reference="${prefix}forearm_link">
+      <material>Gazebo/Blue</material>
+    </gazebo>
+    <gazebo reference="${prefix}wrist_1_link">
+      <material>Gazebo/LightGrey</material>
+    </gazebo>
+    <gazebo reference="${prefix}wrist_2_link">
+      <material>Gazebo/LightGrey</material>
+    </gazebo>
+    <gazebo reference="${prefix}wrist_3_link">
+      <material>Gazebo/LightGrey</material>
+    </gazebo>
+    <!-- ============================================================ -->
+    <!-- Materials -->
+    <!-- ============================================================ -->
+    <material name="Grey">
+      <color rgba="0.5 0.5 0.5 1.0"/>
+    </material>
+    <material name="Blue">
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